Commit message: Updated Robot and Joy Controllers

File: description/camera.xacro (robot description, xacro)
@@ -4,5 +4,5 @@
         <parent link="chassis"/>
         <child link="camera_link"/>
-        <origin xyz="0.305 0 0.08" rpy="0 0 0"/>
+        <origin xyz="0.205 0 0.05" rpy="0 0 0"/>
     </joint>
     <link name="camera_link">

File: description/face.xacro (robot description, xacro)
@@ -8,5 +8,5 @@
     <link name="face_link">
         <visual>
-            <origin xyz="0 0.05 0.01" rpy="0 ${pi/2} 0"/>
+            <origin xyz="-0.1 0.05 0.01" rpy="0 ${pi/2} 0"/>
             <geometry>
                 <cylinder radius="0.01" length="0.002"/>
@@ -15,5 +15,5 @@
         </visual>
         <visual>
-            <origin xyz="0 -0.05 0.01" rpy="0 ${pi/2} 0"/>
+            <origin xyz="-0.1 -0.05 0.01" rpy="0 ${pi/2} 0"/>
             <geometry>
                 <cylinder radius="0.01" length="0.002"/>
@@ -22,5 +22,5 @@
         </visual>
         <visual>
-            <origin xyz="-0.011 0 -0.00" rpy="0 ${1.5} 0"/>
+            <origin xyz="-0.112 0 -0.00" rpy="0 ${1.5} 0"/>
             <geometry>
                 <cylinder radius="0.05" length="0.02"/>

File: description/lidar.xacro (robot description, xacro)
@@ -4,10 +4,10 @@
         <parent link="chassis"/>
         <child link="laser_frame"/>
-        <origin xyz="0.1 0 0.175" rpy="0 0 0"/>
+        <origin xyz="0.040 0 0.1395" rpy="0 0 0"/>
     </joint>
     <link name="laser_frame">
         <visual>
             <geometry>
-                <cylinder radius="0.05" length="0.04"/>
+                <cylinder radius="0.035" length="0.04"/>
             </geometry>
             <material name="red"/>
@@ -18,5 +18,5 @@
             </geometry>
         </collision>
-        <xacro:inertial_cylinder mass="0.1" length="0.04" radius="0.05">
+        <xacro:inertial_cylinder mass="0.2" length="0.04" radius="0.05">
             <origin xyz="0 0 0" rpy="0 0 0"/>
         </xacro:inertial_cylinder>

File: description/robot_core.xacro (robot description, xacro)
@@ -1,142 +1,179 @@
 <?xml version="1.0"?>
-<robot xmlns:xacro="http://www.ros.org/wiki/xacro" >
-    <xacro:include filename="inertial_macros.xacro"/>
-    <xacro:property name="chassis_length" value="0.335"/>
-    <xacro:property name="chassis_width" value="0.265"/>
-    <xacro:property name="chassis_height" value="0.138"/>
-    <xacro:property name="chassis_mass" value="1.0"/>
-    <xacro:property name="wheel_radius" value="0.033"/>
-    <xacro:property name="wheel_thickness" value="0.026"/>
-    <xacro:property name="wheel_mass" value="0.05"/>
-    <xacro:property name="wheel_offset_x" value="0.226"/>
-    <xacro:property name="wheel_offset_y" value="0.1485"/>
-    <xacro:property name="wheel_offset_z" value="0.01"/>
-    <xacro:property name="caster_wheel_radius" value="0.01"/>
-    <xacro:property name="caster_wheel_mass" value="0.01"/>
-    <xacro:property name="caster_wheel_offset_x" value="0.075"/>
-    <xacro:property name="caster_wheel_offset_z" value="${wheel_offset_z - wheel_radius + caster_wheel_radius}"/>
+<robot xmlns:xacro="http://www.ros.org/wiki/xacro">
+    <xacro:include filename="inertial_macros.xacro" />
+    <!-- Robot Properties -->
+    <xacro:property name="chassis_length" value="0.300" />
+    <xacro:property name="chassis_width" value="0.200" />
+    <xacro:property name="chassis_height" value="0.1095" />
+    <xacro:property name="chassis_mass" value="0.5" />
+    <xacro:property name="wheel_radius" value="0.035" />
+    <xacro:property name="wheel_thickness" value="0.0266" />
+    <xacro:property name="wheel_mass" value="0.085" />
+    <xacro:property name="wheel_offset_x" value="0.150" />
+    <xacro:property name="wheel_offset_y" value="0.1233" />
+    <xacro:property name="wheel_offset_z" value="0.035" />
+    <xacro:property name="caster_wheel_radius" value="0.0125" />
+    <xacro:property name="caster_wheel_mass" value="0.05" />
+    <xacro:property name="caster_wheel_offset_x" value="-0.024" />
+    <xacro:property name="caster_wheel_offset_y" value="-0.012" />
+    <xacro:property name="caster_wheel_offset_z" value="-0.058" />
+    <!-- Materials -->
     <material name="white">
         <color rgba="1 1 1 1" />
     </material>
     <material name="orange">
-        <color rgba="1 0.3 0.1 1"/>
+        <color rgba="1 0.3 0.1 1" />
     </material>
     <material name="blue">
-        <color rgba="0.2 0.2 1 1"/>
+        <color rgba="0.2 0.2 1 1" />
     </material>
     <material name="black">
-        <color rgba="0 0 0 1"/>
+        <color rgba="0 0 0 1" />
     </material>
     <material name="red">
-        <color rgba="1 0 0 1"/>
+        <color rgba="1 0 0 1" />
+    </material>
+    <material name="brown">
+        <color rgba="0.65 0.33 0.16 1.0" />
     </material>
     <!-- BASE LINK -->
     <link name="base_link">
+        <inertial>
+            <mass value="1e-6" />
+            <inertia ixx="1e-6" ixy="0" ixz="0" iyy="1e-6" iyz="0" izz="1e-6" />
+        </inertial>
     </link>
     <!-- CHASSIS LINK -->
     <joint name="chassis_joint" type="fixed">
-        <parent link="base_link"/>
-        <child link="chassis"/>
-        <origin xyz="${-wheel_offset_x} 0 ${-wheel_offset_z}"/>
+        <parent link="base_link" />
+        <child link="chassis" />
+        <origin xyz="${-wheel_offset_x} 0 ${wheel_radius}" />
     </joint>
     <link name="chassis">
+        <!-- Main chassis box -->
         <visual>
-            <origin xyz="${chassis_length/2} 0 ${chassis_height/2}"/>
+            <origin xyz="0.1 0 ${chassis_height/2}" />
             <geometry>
-                <box size="${chassis_length} ${chassis_width} ${chassis_height}"/>
+                <box size="0.2 ${chassis_width} ${chassis_height}" />
             </geometry>
-            <material name="orange"/>
+            <material name="brown" />
+        </visual>
+        <!-- Rounded back using cylinder -->
+        <visual>
+            <origin xyz="0 0 ${chassis_height/2}" />
+            <geometry>
+                <cylinder radius="${chassis_width/2}" length="${chassis_height}" />
+            </geometry>
+            <material name="brown" />
         </visual>
         <collision>
-            <origin xyz="${chassis_length/2} 0 ${chassis_height/2}"/>
+            <origin xyz="0.1 0 ${chassis_height/2}" />
             <geometry>
-                <box size="${chassis_length} ${chassis_width} ${chassis_height}"/>
+                <box size="0.2 ${chassis_width} ${chassis_height}" />
             </geometry>
         </collision>
-        <xacro:inertial_box mass="0.5" x="${chassis_length}" y="${chassis_width}" z="${chassis_height}">
-            <origin xyz="${chassis_length/2} 0 ${chassis_height/2}" rpy="0 0 0"/>
+        <collision>
+            <origin xyz="0 0 ${chassis_height/2}" />
+            <geometry>
+                <cylinder radius="${chassis_width/2}" length="${chassis_height}" />
+            </geometry>
+        </collision>
+        <!-- Inertial properties for combined shape -->
+        <xacro:inertial_box mass="${chassis_mass * 0.7}" x="0.2" y="${chassis_width}"
+            z="${chassis_height}">
+            <origin xyz="0.1 0 ${chassis_height/2}" rpy="0 0 0" />
         </xacro:inertial_box>
+        <xacro:inertial_cylinder mass="${chassis_mass * 0.3}" length="${chassis_height}"
+            radius="${chassis_width/2}">
+            <origin xyz="0 0 ${chassis_height/2}" rpy="0 0 0" />
+        </xacro:inertial_cylinder>
     </link>
     <gazebo reference="chassis">
-        <material>Gazebo/Orange</material>
+        <material>Gazebo/Brown</material>
     </gazebo>
     <!-- LEFT WHEEL LINK -->
     <joint name="left_wheel_joint" type="continuous">
-        <parent link="base_link"/>
-        <child link="left_wheel"/>
-        <origin xyz="0 ${wheel_offset_y} 0" rpy="-${pi/2} 0 0" />
-        <axis xyz="0 0 1"/>
+        <parent link="base_link" />  <!-- Keep base_link as parent -->
+        <child link="left_wheel" />
+        <origin xyz="0 ${wheel_offset_y} 0" rpy="-${pi/2} 0 0" /> <!-- Correct orientation -->
+        <axis xyz="0 0 1" />  <!-- Important for correct turning -->
     </joint>
     <link name="left_wheel">
         <visual>
             <geometry>
-                <cylinder radius="${wheel_radius}" length="${wheel_thickness}"/>
+                <cylinder radius="${wheel_radius}" length="${wheel_thickness}" />
             </geometry>
-            <material name="blue"/>
+            <material name="blue" />
         </visual>
         <collision>
             <geometry>
-                <sphere radius="${wheel_radius}"/>
+                <sphere radius="${wheel_radius}" />
             </geometry>
         </collision>
-        <xacro:inertial_cylinder mass="${wheel_mass}" length="${wheel_thickness}" radius="${wheel_radius}">
-            <origin xyz="0 0 0" rpy="0 0 0"/>
+        <xacro:inertial_cylinder mass="${wheel_mass}" length="${wheel_thickness}"
+            radius="${wheel_radius}">
+            <origin xyz="0 0 0" rpy="0 0 0" />
         </xacro:inertial_cylinder>
     </link>
     <gazebo reference="left_wheel">
         <material>Gazebo/Blue</material>
+        <mu1 value="0.9" />
+        <mu2 value="0.9" />
     </gazebo>
     <!-- RIGHT WHEEL LINK -->
     <joint name="right_wheel_joint" type="continuous">
-        <parent link="base_link"/>
-        <child link="right_wheel"/>
-        <origin xyz="0 ${-wheel_offset_y} 0" rpy="${pi/2} 0 0" />
-        <axis xyz="0 0 -1"/>
+        <parent link="base_link" />  <!-- Keep base_link as parent -->
+        <child link="right_wheel" />
+        <origin xyz="0 ${-wheel_offset_y} 0" rpy="${pi/2} 0 0" /> <!-- Correct orientation -->
+        <axis xyz="0 0 -1" />  <!-- Important for correct turning -->
     </joint>
     <link name="right_wheel">
         <visual>
             <geometry>
-                <cylinder radius="${wheel_radius}" length="${wheel_thickness}"/>
+                <cylinder radius="${wheel_radius}" length="${wheel_thickness}" />
             </geometry>
-            <material name="blue"/>
+            <material name="blue" />
         </visual>
         <collision>
             <geometry>
-                <sphere radius="${wheel_radius}"/>
+                <sphere radius="${wheel_radius}" />
             </geometry>
         </collision>
-        <xacro:inertial_cylinder mass="${wheel_mass}" length="${wheel_thickness}" radius="${wheel_radius}">
-            <origin xyz="0 0 0" rpy="0 0 0"/>
+        <xacro:inertial_cylinder mass="${wheel_mass}" length="${wheel_thickness}"
+            radius="${wheel_radius}">
+            <origin xyz="0 0 0" rpy="0 0 0" />
         </xacro:inertial_cylinder>
     </link>
     <gazebo reference="right_wheel">
         <material>Gazebo/Blue</material>
+        <mu1 value="0.9" />
+        <mu2 value="0.9" />
     </gazebo>
     <!-- CASTER WHEEL LINK -->
     <joint name="caster_wheel_joint" type="fixed">
-        <parent link="chassis"/>
-        <child link="caster_wheel"/>
-        <origin xyz="${caster_wheel_offset_x} 0 ${caster_wheel_offset_z}"/>
+        <parent link="chassis" />
+        <child link="caster_wheel" />
+        <origin xyz="${caster_wheel_offset_x} ${caster_wheel_offset_y} ${caster_wheel_offset_z}" />
     </joint>
     <link name="caster_wheel">
         <visual>
             <geometry>
-                <sphere radius="${caster_wheel_radius}"/>
+                <sphere radius="${caster_wheel_radius}" />
             </geometry>
-            <material name="white"/>
+            <material name="white" />
         </visual>
         <collision>
             <geometry>
-                <sphere radius="${caster_wheel_radius}"/>
+                <sphere radius="${caster_wheel_radius}" />
             </geometry>
         </collision>
         <xacro:inertial_sphere mass="${caster_wheel_mass}" radius="${caster_wheel_radius}">
-            <origin xyz="0 0 0" rpy="0 0 0"/>
+            <origin xyz="0 0 0" rpy="0 0 0" />
         </xacro:inertial_sphere>
     </link>
     <gazebo reference="caster_wheel">
         <material>Gazebo/White</material>
-        <mu1 value="0.001"/>
-        <mu2 value="0.001"/>
+        <mu1 value="0.5" />
+        <mu2 value="0.5" />
     </gazebo>
 </robot>

File: description/ros2_control.xacro (robot description, xacro)
@@ -11,5 +11,5 @@
                 <param name="baud_rate">57600</param>
                 <param name="timeout">1000</param>
-                <param name="enc_counts_per_rev">3436</param>
+                <param name="enc_counts_per_rev">3722</param>
             </hardware>
             <joint name="left_wheel_joint">
