Commit message: Created Gazebo Simulation

File: description/robot_core.xacro (robot description, xacro)
@@ -41,4 +41,7 @@
         </xacro:inertial_box>
     </link>
+    <gazebo reference="chassis">
+        <material>Gazebo/White</material>
+    </gazebo>
     <!-- LEFT WHHEL LINK-->
     <joint name="left_wheel_joint" type="continuous">
@@ -64,4 +67,7 @@
         </xacro:inertial_cylinder>
     </link>
+    <gazebo reference="left_wheel">
+        <material>Gazebo/Blue</material>
+    </gazebo>
     <!-- RIGHT WHHEL LINK-->
     <joint name="right_wheel_joint" type="continuous">
@@ -87,4 +93,7 @@
         </xacro:inertial_cylinder>
     </link>
+    <gazebo reference="right_wheel">
+        <material>Gazebo/Blue</material>
+    </gazebo>
     <!-- CASTER WHHEL LINK-->
     <joint name="caster_wheel_joint" type="fixed">
@@ -109,3 +118,8 @@
         </xacro:inertial_sphere>
     </link>
+    <gazebo reference="caster_wheel">
+        <material>Gazebo/Black</material>
+        <mu1 value="0.001"/>
+        <mu2 value="0.001"/>
+    </gazebo>
 </robot>

Commit message: Added Lidar and Motor Controls

File: description/robot_core.xacro (robot description, xacro)
@@ -13,4 +13,7 @@
     <material name="black">
         <color rgba="0 0 0 1" />
+    </material>
+    <material name="red">
+        <color rgba="1 0 0 1" />
     </material>
     <!-- BASE LINK -->

Commit message: Added SLAM config

File: description/robot_core.xacro (robot description, xacro)
@@ -2,21 +2,19 @@
 <robot xmlns:xacro="http://www.ros.org/wiki/xacro">
     <xacro:include filename="inertial_macros.xacro" />
-    <!-- Robot Properties -->
     <xacro:property name="chassis_length" value="0.300" />
     <xacro:property name="chassis_width" value="0.200" />
     <xacro:property name="chassis_height" value="0.1095" />
-    <xacro:property name="chassis_mass" value="0.5" />
+    <xacro:property name="chassis_mass" value="1.5" />
     <xacro:property name="wheel_radius" value="0.035" />
-    <xacro:property name="wheel_thickness" value="0.0266" />
-    <xacro:property name="wheel_mass" value="0.085" />
-    <xacro:property name="wheel_offset_x" value="0.150" />
+    <xacro:property name="wheel_thickness" value="0.026" />
+    <xacro:property name="wheel_mass" value="0.05" />
+    <xacro:property name="wheel_offset_x" value="0.226" />
     <xacro:property name="wheel_offset_y" value="0.1233" />
-    <xacro:property name="wheel_offset_z" value="0.035" />
-    <xacro:property name="caster_wheel_radius" value="0.0125" />
-    <xacro:property name="caster_wheel_mass" value="0.05" />
-    <xacro:property name="caster_wheel_offset_x" value="-0.024" />
-    <xacro:property name="caster_wheel_offset_y" value="-0.012" />
-    <xacro:property name="caster_wheel_offset_z" value="-0.058" />
-    <!-- Materials -->
+    <xacro:property name="wheel_offset_z" value="0.01" />
+    <xacro:property name="caster_wheel_radius" value="0.01" />
+    <xacro:property name="caster_wheel_mass" value="0.01" />
+    <xacro:property name="caster_wheel_offset_x" value="0.060" />
+    <xacro:property name="caster_wheel_offset_z"
+        value="-0.055" />
     <material name="white">
         <color rgba="1 1 1 1" />
@@ -34,13 +32,14 @@
         <color rgba="1 0 0 1" />
     </material>
-    <material name="brown">
-        <color rgba="0.65 0.33 0.16 1.0" />
-    </material>
     <!-- BASE LINK -->
     <link name="base_link">
-        <inertial>
-            <mass value="1e-6" />
-            <inertia ixx="1e-6" ixy="0" ixz="0" iyy="1e-6" iyz="0" izz="1e-6" />
-        </inertial>
+    </link>
+    <!-- BASE_FOOTPRINT_LINK -->
+    <joint name="base_footprint_joint" type="fixed">
+        <parent link="base_link" />
+        <child link="base_footprint" />
+        <origin xyz="0 0 0 " rpy="0 0 0" />
+    </joint>
+    <link name="base_footprint">
     </link>
     <!-- CHASSIS LINK -->
@@ -48,54 +47,34 @@
         <parent link="base_link" />
         <child link="chassis" />
-        <origin xyz="${-wheel_offset_x} 0 ${wheel_radius}" />
+        <origin xyz="${-wheel_offset_x} 0 ${-wheel_offset_z + wheel_radius + 0.005}" />
     </joint>
     <link name="chassis">
-        <!-- Main chassis box -->
         <visual>
-            <origin xyz="0.1 0 ${chassis_height/2}" />
+            <origin xyz="${chassis_length/2} 0 ${chassis_height/2}" />
             <geometry>
-                <box size="0.2 ${chassis_width} ${chassis_height}" />
+                <box size="${chassis_length} ${chassis_width} ${chassis_height}" />
             </geometry>
-            <material name="brown" />
-        </visual>
-        <!-- Rounded back using cylinder -->
-        <visual>
-            <origin xyz="0 0 ${chassis_height/2}" />
-            <geometry>
-                <cylinder radius="${chassis_width/2}" length="${chassis_height}" />
-            </geometry>
-            <material name="brown" />
+            <material name="orange" />
         </visual>
         <collision>
-            <origin xyz="0.1 0 ${chassis_height/2}" />
+            <origin xyz="${chassis_length/2} 0 ${chassis_height/2}" />
             <geometry>
-                <box size="0.2 ${chassis_width} ${chassis_height}" />
+                <box size="${chassis_length} ${chassis_width} ${chassis_height}" />
             </geometry>
         </collision>
-        <collision>
-            <origin xyz="0 0 ${chassis_height/2}" />
-            <geometry>
-                <cylinder radius="${chassis_width/2}" length="${chassis_height}" />
-            </geometry>
-        </collision>
-        <!-- Inertial properties for combined shape -->
-        <xacro:inertial_box mass="${chassis_mass * 0.7}" x="0.2" y="${chassis_width}"
+        <xacro:inertial_box mass="0.5" x="${chassis_length}" y="${chassis_width}"
             z="${chassis_height}">
-            <origin xyz="0.1 0 ${chassis_height/2}" rpy="0 0 0" />
+            <origin xyz="${chassis_length/2} 0 ${chassis_height/2}" rpy="0 0 0" />
         </xacro:inertial_box>
-        <xacro:inertial_cylinder mass="${chassis_mass * 0.3}" length="${chassis_height}"
-            radius="${chassis_width/2}">
-            <origin xyz="0 0 ${chassis_height/2}" rpy="0 0 0" />
-        </xacro:inertial_cylinder>
     </link>
     <gazebo reference="chassis">
-        <material>Gazebo/Brown</material>
+        <material>Gazebo/Orange</material>
     </gazebo>
     <!-- LEFT WHEEL LINK -->
     <joint name="left_wheel_joint" type="continuous">
-        <parent link="base_link" />  <!-- Keep base_link as parent -->
+        <parent link="base_link" />
         <child link="left_wheel" />
-        <origin xyz="0 ${wheel_offset_y} 0" rpy="-${pi/2} 0 0" /> <!-- Correct orientation -->
-        <axis xyz="0 0 1" />  <!-- Important for correct turning -->
+        <origin xyz="0 ${wheel_offset_y} 0" rpy="-${pi/2} 0 0" />
+        <axis xyz="0 0 1" />
     </joint>
     <link name="left_wheel">
@@ -118,13 +97,11 @@
     <gazebo reference="left_wheel">
         <material>Gazebo/Blue</material>
-        <mu1 value="0.9" />
-        <mu2 value="0.9" />
     </gazebo>
     <!-- RIGHT WHEEL LINK -->
     <joint name="right_wheel_joint" type="continuous">
-        <parent link="base_link" />  <!-- Keep base_link as parent -->
+        <parent link="base_link" />
         <child link="right_wheel" />
-        <origin xyz="0 ${-wheel_offset_y} 0" rpy="${pi/2} 0 0" /> <!-- Correct orientation -->
-        <axis xyz="0 0 -1" />  <!-- Important for correct turning -->
+        <origin xyz="0 ${-wheel_offset_y} 0" rpy="${pi/2} 0 0" />
+        <axis xyz="0 0 -1" />
     </joint>
     <link name="right_wheel">
@@ -147,6 +124,4 @@
     <gazebo reference="right_wheel">
         <material>Gazebo/Blue</material>
-        <mu1 value="0.9" />
-        <mu2 value="0.9" />
     </gazebo>
     <!-- CASTER WHEEL LINK -->
@@ -154,5 +129,5 @@
         <parent link="chassis" />
         <child link="caster_wheel" />
-        <origin xyz="${caster_wheel_offset_x} ${caster_wheel_offset_y} ${caster_wheel_offset_z}" />
+        <origin xyz="${caster_wheel_offset_x} 0 ${caster_wheel_offset_z}" />
     </joint>
     <link name="caster_wheel">
@@ -174,6 +149,6 @@
     <gazebo reference="caster_wheel">
         <material>Gazebo/White</material>
-        <mu1 value="0.5" />
-        <mu2 value="0.5" />
+        <mu1 value="0.001" />
+        <mu2 value="0.001" />
     </gazebo>
 </robot>
